File: PCB/board.kicad_pcb (KiCad board)
At the start: 2 copper layers, 42.4 x 61.4 mm, 5 parts, among them SW1 SW_Push, SW2 SW_Push, SW3 SW_Push, SW4 SW_Push, U1 MOUDLE-SEEEDUINO-XIAO

Commit message: Add firmware
Connections:
- SW2 pad 1: GND -> Net-(U1-PA4_A1_D1)
- SW2 pad 2: Net-(U1-PA4_A1_D1) -> GND
Routing:
- net GND: track 103.4 -> 0.00 mm
- net Net-(U1-PA4_A1_D1): track 25.0 -> 40.7 mm
- net Net-(U1-PA11_A3_D3): track 55.9 -> 47.7 mm
- net Net-(U1-PA10_A2_D2): track 36.9 -> 43.1 mm
- net Net-(U1-PA02_A0_D0): track 31.8 -> 26.9 mm
- added copper zone on B.Cu, net GND
- added copper zone on F.Cu, net GND
Changed lines of the file:
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@@
 			(layers "*.Cu" "*.Mask")
 			(remove_unused_layers no)
-			(net "GND")
+			(net "Net-(U1-PA4_A1_D1)")
 			(pinfunction "1_1")
 			(pintype "passive")
@@
 			(layers "*.Cu" "*.Mask")
 			(remove_unused_layers no)
-			(net "Net-(U1-PA4_A1_D1)")
+			(net "GND")
 			(pinfunction "2_2")
 			(pintype "passive")
@@
 			(net "unconnected-(U1-PA8_A4_D4_SDA-Pad5)")
 			(pinfunction "PA8_A4_D4_SDA_5")
-			(pintype "passive")
+			(pintype "passive+no_connect")
 		)
 		(pad "6" thru_hole oval
@@
 			(net "unconnected-(U1-PA9_A5_D5_SCL-Pad6)")
 			(pinfunction "PA9_A5_D5_SCL_6")
-			(pintype "passive")
+			(pintype "passive+no_connect")
 		)
 		(pad "7" thru_hole oval
@@
 			(net "unconnected-(U1-PB08_A6_D6_TX-Pad7)")
 			(pinfunction "PB08_A6_D6_TX_7")
-			(pintype "passive")
+			(pintype "passive+no_connect")
 		)
 		(pad "8" thru_hole oval
@@
 			(net "unconnected-(U1-PB09_A7_D7_RX-Pad8)")
 			(pinfunction "PB09_A7_D7_RX_8")
-			(pintype "passive")
+			(pintype "passive+no_connect")
 		)
 		(pad "9" thru_hole oval
@@
 			(net "unconnected-(U1-PA7_A8_D8_SCK-Pad9)")
 			(pinfunction "PA7_A8_D8_SCK_9")
-			(pintype "passive")
+			(pintype "passive+no_connect")
 		)
 		(pad "10" thru_hole oval
@@
 			(net "unconnected-(U1-PA5_A9_D9_MISO-Pad10)")
 			(pinfunction "PA5_A9_D9_MISO_10")
-			(pintype "passive")
+			(pintype "passive+no_connect")
 		)
 		(pad "11" thru_hole oval
@@
 			(net "unconnected-(U1-PA6_A10_D10_MOSI-Pad11)")
 			(pinfunction "PA6_A10_D10_MOSI_11")
-			(pintype "passive")
+			(pintype "passive+no_connect")
 		)
 		(pad "12" thru_hole oval
@@
 			(net "unconnected-(U1-3V3-Pad12)")
 			(pinfunction "3V3_12")
-			(pintype "passive")
+			(pintype "passive+no_connect")
 		)
 		(pad "13" thru_hole oval
@@
 			(net "unconnected-(U1-5V-Pad14)")
 			(pinfunction "5V_14")
-			(pintype "passive")
+			(pintype "passive+no_connect")
 		)
 		(embedded_fonts no)
@@
 	)
 	(segment
-		(start 97 90)
-		(end 96 89)
+		(start 89.74 109.665585)
+		(end 92.374415 112.3)
 		(width 0.2)
 		(layer "F.Cu")
-		(net "GND")
+		(net "Net-(U1-PA11_A3_D3)")
 	)
 	(segment
-		(start 105.55 100.003654)
-		(end 105.55 91.960101)
+		(start 80.75 94.08)
+		(end 89.74 103.07)
 		(width 0.2)
 		(layer "F.Cu")
-		(net "GND")
+		(net "Net-(U1-PA11_A3_D3)")
 	)
 	(segment
-		(start 105.55 91.960101)
-		(end 102.589899 89)
+		(start 92.374415 112.3)
+		(end 94.8 112.3)
 		(width 0.2)
 		(layer "F.Cu")
-		(net "GND")
+		(net "Net-(U1-PA11_A3_D3)")
 	)
 	(segment
-		(start 104.15 130.54)
-		(end 111.079899 123.610101)
+		(start 94.8 112.3)
+		(end 110.5 128)
 		(width 0.2)
 		(layer "F.Cu")
-		(net "GND")
+		(net "Net-(U1-PA11_A3_D3)")
 	)
 	(segment
-		(start 111.9 106.353654)
-		(end 105.55 100.003654)
+		(start 89.74 103.07)
+		(end 89.74 109.665585)
 		(width 0.2)
 		(layer "F.Cu")
-		(net "GND")
+		(net "Net-(U1-PA11_A3_D3)")
 	)
 	(segment
-		(start 110.5 90)
-		(end 97 90)
+		(start 91.54 97.25)
+		(end 91.54 108.92)
 		(width 0.2)
 		(layer "F.Cu")
-		(net "GND")
+		(net "Net-(U1-PA02_A0_D0)")
 	)
 	(segment
-		(start 111.079899 110.32)
-		(end 111.9 109.499899)
+		(start 80.75 86.46)
+		(end 91.54 97.25)
 		(width 0.2)
 		(layer "F.Cu")
-		(net "GND")
+		(net "Net-(U1-PA02_A0_D0)")
 	)
 	(segment
-		(start 104.15 111.46)
-		(end 109.939899 111.46)
+		(start 90.14 100.93)
+		(end 90.14 109.499899)
 		(width 0.2)
 		(layer "F.Cu")
-		(net "GND")
+		(net "Net-(U1-PA10_A2_D2)")
 	)
 	(segment
-		(start 111.9 109.499899)
-		(end 111.9 106.353654)
+		(start 90.14 109.499899)
+		(end 90.960101 110.32)
 		(width 0.2)
 		(layer "F.Cu")
-		(net "GND")
+		(net "Net-(U1-PA10_A2_D2)")
 	)
 	(segment
-		(start 109.939899 111.46)
-		(end 111.9 109.499899)
+		(start 104.710101 108.92)
+		(end 110.5 108.92)
 		(width 0.2)
 		(layer "F.Cu")
-		(net "GND")
+		(net "Net-(U1-PA10_A2_D2)")
 	)
 	(segment
-		(start 111.079899 123.610101)
-		(end 111.079899 110.32)
+		(start 90.960101 110.32)
+		(end 103.310101 110.32)
 		(width 0.2)
 		(layer "F.Cu")
-		(net "GND")
+		(net "Net-(U1-PA10_A2_D2)")
 	)
 	(segment
-		(start 102.589899 89)
-		(end 96 89)
+		(start 103.310101 110.32)
+		(end 104.710101 108.92)
 		(width 0.2)
 		(layer "F.Cu")
-		(net "GND")
+		(net "Net-(U1-PA10_A2_D2)")
 	)
 	(segment
-		(start 85.19 111.46)
-		(end 109.939899 111.46)
+		(start 80.75 91.54)
+		(end 90.14 100.93)
 		(width 0.2)
 		(layer "F.Cu")
-		(net "GND")
+		(net "Net-(U1-PA10_A2_D2)")
 	)
 	(segment
-		(start 104.15 92.54)
-		(end 104 92.69)
+		(start 77.7 87.61)
+		(end 77.7 85.31)
 		(width 0.2)
 		(layer "F.Cu")
@@
 	)
 	(segment
-		(start 104 92.69)
-		(end 84.44 92.69)
+		(start 80.75 89)
+		(end 79.09 89)
 		(width 0.2)
 		(layer "F.Cu")
@@
 	)
 	(segment
-		(start 84.44 92.69)
-		(end 80.75 89)
+		(start 79.09 89)
+		(end 77.7 87.61)
 		(width 0.2)
 		(layer "F.Cu")
@@
 	)
 	(segment
-		(start 110.5 128)
-		(end 108.669899 128)
-		(width 0.2)
-		(layer "F.Cu")
-		(net "Net-(U1-PA11_A3_D3)")
-	)
-	(segment
-		(start 81.96033 110.330229)
-		(end 81.96033 95.29033)
-		(width 0.2)
-		(layer "F.Cu")
-		(net "Net-(U1-PA11_A3_D3)")
-	)
-	(segment
-		(start 81.96033 95.29033)
-		(end 80.75 94.08)
-		(width 0.2)
-		(layer "F.Cu")
-		(net "Net-(U1-PA11_A3_D3)")
-	)
-	(segment
-		(start 103.570101 131.94)
-		(end 81.96033 110.330229)
-		(width 0.2)
-		(layer "F.Cu")
-		(net "Net-(U1-PA11_A3_D3)")
-	)
-	(segment
-		(start 108.669899 128)
-		(end 104.729899 131.94)
-		(width 0.2)
-		(layer "F.Cu")
-		(net "Net-(U1-PA11_A3_D3)")
-	)
-	(segment
-		(start 104.729899 131.94)
-		(end 103.570101 131.94)
-		(width 0.2)
-		(layer "F.Cu")
-		(net "Net-(U1-PA11_A3_D3)")
-	)
-	(segment
-		(start 91.54 108.92)
-		(end 91.54 103.053654)
-		(width 0.2)
-		(layer "F.Cu")
-		(net "Net-(U1-PA02_A0_D0)")
-	)
-	(segment
-		(start 78.323654 92.69)
-		(end 77.65 92.016346)
-		(width 0.2)
-		(layer "F.Cu")
-		(net "Net-(U1-PA02_A0_D0)")
-	)
-	(segment
-		(start 79.713654 86.46)
-		(end 80.75 86.46)
-		(width 0.2)
-		(layer "F.Cu")
-		(net "Net-(U1-PA02_A0_D0)")
-	)
-	(segment
-		(start 77.65 88.523654)
-		(end 79.713654 86.46)
+		(start 105.81 85.31)
+		(end 110.5 90)
 		(width 0.2)
 		(layer "F.Cu")
-		(net "Net-(U1-PA02_A0_D0)")
-	)
-	(segment
-		(start 91.54 103.053654)
-		(end 81.176346 92.69)
-		(width 0.2)
-		(layer "F.Cu")
-		(net "Net-(U1-PA02_A0_D0)")
-	)
-	(segment
-		(start 81.176346 92.69)
-		(end 78.323654 92.69)
-		(width 0.2)
-		(layer "F.Cu")
-		(net "Net-(U1-PA02_A0_D0)")
-	)
-	(segment
-		(start 77.65 92.016346)
-		(end 77.65 88.523654)
-		(width 0.2)
-		(layer "F.Cu")
-		(net "Net-(U1-PA02_A0_D0)")
+		(net "Net-(U1-PA4_A1_D1)")
 	)
 	(segment
-		(start 110.5 108.92)
-		(end 98.13 108.92)
+		(start 77.7 85.31)
+		(end 105.81 85.31)
 		(width 0.2)
 		(layer "F.Cu")
-		(net "Net-(U1-PA10_A2_D2)")
+		(net "Net-(U1-PA4_A1_D1)")
 	)
-	(segment
-		(start 98.13 108.92)
-		(end 80.75 91.54)
-		(width 0.2)
-		(layer "F.Cu")
-		(net "Net-(U1-PA10_A2_D2)")
+	(zone
+		(net "GND")
+		(layers "F.Cu" "B.Cu")
+		(name "GND")
+		(hatch edge 0.5)
+		(connect_pads
+			(clearance 0.5)
+		)
+		(min_thickness 0.25)
+		(fill yes
+			(thermal_gap 0.5)
+			(thermal_bridge_width 0.5)
+			(island_removal_mode 0)
+		)
+		(polygon
+			(pts
+				(xy 71.85 79.95) (xy 122.55 81.45) (xy 127.75 151.6) (xy 62.55 152.9)
+			)
+		)
 	)
 	(embedded_fonts no)

Commit message: Syncing it with local clone
Other:
- board size 42.4 x 61.4 mm -> 40.6 x 59.2 mm
Changed lines of the file:
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@@
 		)
 		(embedded_fonts no)
-		(model "${KICAD10_3DMODEL_DIR}/Button_Switch_Keyboard.3dshapes/SW_Cherry_MX_1.00u_PCB.step"
+		(model "${KIPRJMOD}/MX .STEP"
 			(offset
-				(xyz 0 0 0)
+				(xyz 4.8 2.25 4.5)
 			)
 			(scale
@@
 			)
 			(rotate
-				(xyz 0 0 0)
+				(xyz -90 -0 -180)
+			)
+		)
+		(model "${KIPRJMOD}/DSA_Keycap_CherryMX.step"
+			(offset
+				(xyz -2 -4.5 10)
+			)
+			(scale
+				(xyz 1 1 1)
+			)
+			(rotate
+				(xyz -90 -0 -0)
 			)
 		)
@@
 		)
 		(embedded_fonts no)
-		(model "${KICAD10_3DMODEL_DIR}/Button_Switch_Keyboard.3dshapes/SW_Cherry_MX_1.00u_PCB.step"
+		(model "${KIPRJMOD}/MX .STEP"
+			(offset
+				(xyz 4.8 2.25 4.5)
+			)
+			(scale
+				(xyz 1 1 1)
+			)
+			(rotate
+				(xyz -90 -0 -180)
+			)
+		)
+		(model "${KIPRJMOD}/DSA_Keycap_CherryMX.step"
 			(offset
-				(xyz 0 0 0)
+				(xyz -2 -4.5 10)
 			)
 			(scale
@@
 			)
 			(rotate
-				(xyz 0 0 0)
+				(xyz -90 -0 -0)
 			)
 		)
@@
 		)
 		(embedded_fonts no)
-		(model "${KICAD10_3DMODEL_DIR}/Button_Switch_Keyboard.3dshapes/SW_Cherry_MX_1.00u_PCB.step"
+		(model "${KIPRJMOD}/DSA_Keycap_CherryMX.step"
+			(offset
+				(xyz -2 -4.5 9.5)
+			)
+			(scale
+				(xyz 1 1 1)
+			)
+			(rotate
+				(xyz -90 -0 -0)
+			)
+		)
+		(model "${KIPRJMOD}/MX .STEP"
 			(offset
-				(xyz 0 0 0)
+				(xyz 4.8 2.25 4.5)
 			)
 			(scale
@@
 			)
 			(rotate
-				(xyz 0 0 0)
+				(xyz -90 -0 -180)
 			)
 		)
@@
 		)
 		(embedded_fonts no)
+		(model "${KIPRJMOD}/Seeed Studio XIAO RP2040 v26 v2 (1).step"
+			(offset
+				(xyz 0 0 2.5)
+			)
+			(scale
+				(xyz 1 1 1)
+			)
+			(rotate
+				(xyz -0 -0 -0)
+			)
+		)
 	)
 	(footprint "Button_Switch_Keyboard:SW_Cherry_MX_1.00u_PCB"
@@
 		)
 		(embedded_fonts no)
-		(model "${KICAD10_3DMODEL_DIR}/Button_Switch_Keyboard.3dshapes/SW_Cherry_MX_1.00u_PCB.step"
+		(model "${KIPRJMOD}/DSA_Keycap_CherryMX.step"
+			(offset
+				(xyz -2 -4.5 9.5)
+			)
+			(scale
+				(xyz 1 1 1)
+			)
+			(rotate
+				(xyz -90 -0 -0)
+			)
+		)
+		(model "${KIPRJMOD}/MX .STEP"
 			(offset
-				(xyz 0 0 0)
+				(xyz 4.8 2.25 4.5)
 			)
 			(scale
@@
 			)
 			(rotate
-				(xyz 0 0 0)
+				(xyz -90 -0 180)
 			)
 		)
 	)
 	(gr_rect
-		(start 75.635876 83.144564)
-		(end 118 144.5)
+		(start 77 83.52)
+		(end 117.6 142.72)
+		(radius 1)
 		(stroke
 			(width 0.05)
@@
 	)
 	(gr_text "aditya\n"
-		(at 91.5 144.5 90)
+		(at 91.6 143.29 90)
 		(layer "F.SilkS")
 		(effects
 			(font
-				(size 4.5 4.5)
-				(thickness 0.25)
+				(size 4.5 4.2)
+				(thickness 0.9)
+				(bold yes)
 			)
 			(justify left bottom)
@@
 	)
 	(segment
+		(start 77.7 87.61)
+		(end 77.7 85.31)
+		(width 0.2)
+		(layer "F.Cu")
+		(net "Net-(U1-PA4_A1_D1)")
+	)
+	(segment
+		(start 80.75 89)
+		(end 79.09 89)
+		(width 0.2)
+		(layer "F.Cu")
+		(net "Net-(U1-PA4_A1_D1)")
+	)
+	(segment
+		(start 79.09 89)
+		(end 77.7 87.61)
+		(width 0.2)
+		(layer "F.Cu")
+		(net "Net-(U1-PA4_A1_D1)")
+	)
+	(segment
+		(start 105.81 85.31)
+		(end 110.5 90)
+		(width 0.2)
+		(layer "F.Cu")
+		(net "Net-(U1-PA4_A1_D1)")
+	)
+	(segment
+		(start 77.7 85.31)
+		(end 105.81 85.31)
+		(width 0.2)
+		(layer "F.Cu")
+		(net "Net-(U1-PA4_A1_D1)")
+	)
+	(segment
 		(start 89.74 109.665585)
 		(end 92.374415 112.3)
@@
 		(net "Net-(U1-PA10_A2_D2)")
 	)
-	(segment
-		(start 77.7 87.61)
-		(end 77.7 85.31)
-		(width 0.2)
-		(layer "F.Cu")
-		(net "Net-(U1-PA4_A1_D1)")
-	)
-	(segment
-		(start 80.75 89)
-		(end 79.09 89)
-		(width 0.2)
-		(layer "F.Cu")
-		(net "Net-(U1-PA4_A1_D1)")
-	)
-	(segment
-		(start 79.09 89)
-		(end 77.7 87.61)
-		(width 0.2)
-		(layer "F.Cu")
-		(net "Net-(U1-PA4_A1_D1)")
-	)
-	(segment
-		(start 105.81 85.31)
-		(end 110.5 90)
-		(width 0.2)
-		(layer "F.Cu")
-		(net "Net-(U1-PA4_A1_D1)")
-	)
-	(segment
-		(start 77.7 85.31)
-		(end 105.81 85.31)
-		(width 0.2)
-		(layer "F.Cu")
-		(net "Net-(U1-PA4_A1_D1)")
-	)
 	(zone
